File: Daughterboards/Simple/Simple.kicad_sch (KiCad schematic)
At the start: 23 parts, among them J1 I2C EXT, J2 HRO-TYPEC-M12, J3 BATTERY JST, J6 FFC, J7 DEBUG, M1 M.2_Key_E, U4 XC6206P332MR

Commit message: prettify files a lil bit
Parts:
- U1: value (none) -> SRV05-4; footprint (none) -> Package_TO_SOT_SMD:SOT-23-6
Changed lines of the file:
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@@
       (effects (font (size 1.27 1.27)) (justify left))
     )
-    (property "Value" "" (id 1) (at 167.2337 38.735 0)
+    (property "Value" "SRV05-4" (id 1) (at 167.2337 38.735 0)
       (effects (font (size 1.27 1.27)) (justify left))
     )
-    (property "Footprint" "" (id 2) (at 182.245 62.865 0)
+    (property "Footprint" "Package_TO_SOT_SMD:SOT-23-6" (id 2) (at 182.245 62.865 0)
       (effects (font (size 1.27 1.27)) hide)
     )
